Commit message: Update so101 urdf and srdf

File: src/SO101/so101_brush_tip_nominal.urdf (robot description, URDF)
Before this commit: robot so101_new_calib, 11 links, 10 joints
Links:
- added link arm_mount; collision mesh filename=assets/arm_base.stl scale=0.001 0.001 0.001; visual mesh filename=assets/arm_base.stl scale=0.001 0.001 0.001
- added link table; collision box size=1.5 1.5 0.04; visual box size=1.5 1.5 0.04
Joints:
- added joint base_to_arm_mount: type fixed, parent base_link, child arm_mount, origin xyz=0.072956211 -0.053430466 -0.0024 rpy=1.5707963267948966 0 0
- added joint base_to_table: type fixed, parent base_link, child table, origin xyz=0 0 -0.0274 rpy=0 0 0
